Commit message: Robot does not look wonky and it seems promising to control! :)

File: src/ros_experimenting/models/katana_test.urdf (robot description, URDF)
Before this commit: robot katana_450_6m90a, 10 links, 9 joints
Links:
- added link world
Joints:
- added joint fixed: type fixed, parent world, child katana_base_link
