Commit message: No longer broken

File: src/ros_experimenting/models/BERT2.xacro (robot description, xacro)
@@ -3,6 +3,5 @@
     <!-- Constants for robot dimensions -->
     <xacro:property name="PI" value="3.1415926535897931"/>
-    <xacro:property name="link1_mass" value="2.35" />
-    <xacro:property name="link2_mass" value="3.0" />
+    <xacro:property name="mass" value="2.35" />
     <xacro:property name="width" value="0.1" /> <!-- Square dimensions (widthxwidth) of beams -->
     <xacro:property name="height1" value="2" /> <!-- Link 1 -->
@@ -33,9 +32,9 @@
         <inertial>
             <origin xyz="0 0 ${height1/2}" rpy="0 0 0"/>
-            <link1_mass value="${link1_mass}"/>
+            <mass value="${mass}"/>
             <inertia
-                ixx="${link1_mass / 12.0 * (width*width + height1*height1)}" ixy="0.0" ixz="0.0"
-                iyy="${link1_mass / 12.0 * (height1*height1 + width*width)}" iyz="0.0"
-                izz="${link1_mass / 12.0 * (width*width + width*width)}"/>
+                ixx="${mass / 12.0 * (width*width + height1*height1)}" ixy="0.0" ixz="0.0"
+                iyy="${mass / 12.0 * (height1*height1 + width*width)}" iyz="0.0"
+                izz="${mass / 12.0 * (width*width + width*width)}"/>
         </inertial>
     </link>
@@ -64,9 +63,9 @@
         <inertial>
             <origin xyz="0 0 ${height2/2 - axel_offset}" rpy="0 0 0"/>
-            <link1_mass value="${link1_mass}"/>
+            <mass value="${mass}"/>
             <inertia
-                ixx="${link1_mass / 12.0 * (width*width + height2*height2)}" ixy="0.0" ixz="0.0"
-                iyy="${link1_mass / 12.0 * (height2*height2 + width*width)}" iyz="0.0"
-                izz="${link1_mass / 12.0 * (width*width + width*width)}"/>
+                ixx="${mass / 12.0 * (width*width + height2*height2)}" ixy="0.0" ixz="0.0"
+                iyy="${mass / 12.0 * (height2*height2 + width*width)}" iyz="0.0"
+                izz="${mass / 12.0 * (width*width + width*width)}"/>
         </inertial>
     </link>
@@ -95,9 +94,9 @@
         <inertial>
             <origin xyz="0 0 ${height3/2 - axel_offset}" rpy="0 0 0"/>
-            <link1_mass value="${link1_mass}"/>
+            <mass value="${mass}"/>
             <inertia
-                ixx="${link1_mass / 12.0 * (width*width + height3*height3)}" ixy="0.0" ixz="0.0"
-                iyy="${link1_mass / 12.0 * (height3*height3 + width*width)}" iyz="0.0"
-                izz="${link1_mass / 12.0 * (width*width + width*width)}"/>
+                ixx="${mass / 12.0 * (width*width + height3*height3)}" ixy="0.0" ixz="0.0"
+                iyy="${mass / 12.0 * (height3*height3 + width*width)}" iyz="0.0"
+                izz="${mass / 12.0 * (width*width + width*width)}"/>
         </inertial>
     </link>

Commit message: BERT looks good, need to update inertial

File: src/ros_experimenting/models/BERT2.xacro (robot description, xacro)
@@ -3,18 +3,24 @@
     <!-- Constants for robot dimensions -->
     <xacro:property name="PI" value="3.1415926535897931"/>
-    <xacro:property name="mass" value="2.35" />
+    <xacro:property name="link1_mass" value="2.35" />
+    <xacro:property name="link2_mass" value="3.0" />
+    <xacro:property name="link1_radius" value="0.05" />
+    <xacro:property name="link2_radius" value="0.05" />
+    <xacro:property name="link1_length" value="0.2735" />
+    <xacro:property name="link2_length" value="0.44" />
+    <xacro:property name="mass" value="5" />
+    <xacro:property name="axel_offset" value="0.025" /> <!-- Space btw top of beam and the each joint -->
     <xacro:property name="width" value="0.1" /> <!-- Square dimensions (widthxwidth) of beams -->
     <xacro:property name="height1" value="2" /> <!-- Link 1 -->
     <xacro:property name="height2" value="1" /> <!-- Link 2 -->
     <xacro:property name="height3" value="1" /> <!-- Link 3 -->
-    <xacro:property name="axel_offset" value="0.05" /> <!-- Space btw top of beam and the each joint -->
     <!-- Make the robot's base immovable -->
     <link name="world"/>
     <joint name="fixed" type="fixed">
         <parent link="world"/>
-        <child link="BERT2_link1"/>
+        <child link="BERT2_baselink"/>
     </joint>
     <!-- Base Link -->
-    <link name="BERT2_link1">
+    <link name="BERT2_baselink">
         <collision>
             <origin xyz="0 0 ${height1/2}" rpy="0 0 0"/>
@@ -40,38 +46,38 @@
     </link>
     <joint name="BERT2_joint1" type="continuous">
-        <parent link="BERT2_link1"/>
-        <child link="BERT2_link2"/>
-        <origin xyz="0 ${width} ${height1 - axel_offset}" rpy="0 0 0"/>
+        <parent link="BERT2_baselink"/>
+        <child link="BERT2_link1"/>
+        <origin xyz="0 ${link1_radius*2} ${height1 - axel_offset}" rpy="0 0 0"/>
         <axis xyz="0 1 0"/>
         <dynamics damping="0.7"/>
     </joint>
     <!-- Middle Link -->
-    <link name="BERT2_link2">
+    <link name="BERT2_link1">
         <collision>
-            <origin xyz="0 0 ${height2/2 - axel_offset}" rpy="0 0 0"/>
+            <origin xyz="0 0 ${link1_length/2 - axel_offset}" rpy="0 0 0"/>
             <geometry>
-                <box size="${width} ${width} ${height2}"/>
+                <cylinder radius="${link1_radius}" length="${link1_length}"/>
             </geometry>
         </collision>
         <visual>
-            <origin xyz="0 0 ${height2/2 - axel_offset}" rpy="0 0 0"/>
+            <origin xyz="0 0 ${link1_length/2 - axel_offset}" rpy="0 0 0"/>
             <geometry>
-                <box size="${width} ${width} ${height2}"/>
+                <cylinder radius="${link1_radius}" length="${link1_length}"/>
             </geometry>
             <material name="grey"/>
         </visual>
         <inertial>
-            <origin xyz="0 0 ${height2/2 - axel_offset}" rpy="0 0 0"/>
-            <mass value="${mass}"/>
+            <origin xyz="0 0 ${link1_length/2 - axel_offset}" rpy="0 0 0"/>
+            <mass value="${link1_mass}"/>
             <inertia
-                ixx="${mass / 12.0 * (width*width + height2*height2)}" ixy="0.0" ixz="0.0"
-                iyy="${mass / 12.0 * (height2*height2 + width*width)}" iyz="0.0"
-                izz="${mass / 12.0 * (width*width + width*width)}"/>
+                ixx="${link1_mass / 12.0 * (width*width + height2*height2)}" ixy="0.0" ixz="0.0"
+                iyy="${link1_mass / 12.0 * (height2*height2 + width*width)}" iyz="0.0"
+                izz="${link1_mass / 12.0 * (width*width + width*width)}"/>
         </inertial>
     </link>
     <joint name="BERT2_joint2" type="continuous">
-        <parent link="BERT2_link2"/>
+        <parent link="BERT2_link1"/>
         <child link="BERT2_link3"/>
-        <origin xyz="0 ${width} ${height2 - axel_offset*2}" rpy="0 0 0"/>
+        <origin xyz="0 ${link2_radius*2} ${link1_length - axel_offset*2}" rpy="0 0 0"/>
         <axis xyz="0 1 0"/>
         <dynamics damping="0.7"/>
@@ -80,23 +86,23 @@
     <link name="BERT2_link3">
         <collision>
-            <origin xyz="0 0 ${height3/2 - axel_offset}" rpy="0 0 0"/>
+            <origin xyz="0 0 ${link2_length/2 - axel_offset}" rpy="0 0 0"/>
             <geometry>
-                <box size="${width} ${width} ${height3}"/>
+                <cylinder radius="${link2_radius}" length="${link2_length}"/>
             </geometry>
         </collision>
         <visual>
-            <origin xyz="0 0 ${height3/2 - axel_offset}" rpy="0 0 0"/>
+            <origin xyz="0 0 ${link2_length/2 - axel_offset}" rpy="0 0 0"/>
             <geometry>
-                <box size="${width} ${width} ${height3}"/>
+                <cylinder radius="${link2_radius}" length="${link2_length}"/>
             </geometry>
             <material name="black"/>
         </visual>
         <inertial>
-            <origin xyz="0 0 ${height3/2 - axel_offset}" rpy="0 0 0"/>
-            <mass value="${mass}"/>
+            <origin xyz="0 0 ${link2_length/2 - axel_offset}" rpy="0 0 0"/>
+            <mass value="${link2_mass}"/>
             <inertia
-                ixx="${mass / 12.0 * (width*width + height3*height3)}" ixy="0.0" ixz="0.0"
-                iyy="${mass / 12.0 * (height3*height3 + width*width)}" iyz="0.0"
-                izz="${mass / 12.0 * (width*width + width*width)}"/>
+                ixx="${link2_mass / 12.0 * (width*width + height3*height3)}" ixy="0.0" ixz="0.0"
+                iyy="${link2_mass / 12.0 * (height3*height3 + width*width)}" iyz="0.0"
+                izz="${link2_mass / 12.0 * (width*width + width*width)}"/>
         </inertial>
     </link>
@@ -123,5 +129,5 @@
     </transmission>
     <!-- Gazebo Plugins -->
-    <gazebo>
+    <!-- <gazebo>
         <plugin name="gazebo_ros_control" filename="libgazebo_ros_control.so">
             <robotNamespace>/BERT2_robot</robotNamespace>
@@ -129,10 +135,10 @@
             <controlPeriod>0.01</controlPeriod>
         </plugin>
-    </gazebo>
+    </gazebo> -->
     <!-- Additional Configs -->
-    <gazebo reference="BERT2_link1">
+    <gazebo reference="BERT2_baselink">
         <material>Gazebo/Black</material>
     </gazebo>
-    <gazebo reference="BERT2_link2">
+    <gazebo reference="BERT2_link1">
         <mu1>0.2</mu1>
         <mu2>0.2</mu2>

Commit message: Cleanup xacro naming and putting the initial estimates in the cpp file

File: src/ros_experimenting/models/BERT2.xacro (robot description, xacro)
@@ -78,5 +78,5 @@
     <joint name="BERT2_joint2" type="continuous">
         <parent link="BERT2_link1"/>
-        <child link="BERT2_link3"/>
+        <child link="BERT2_link2"/>
         <origin xyz="0 ${link2_radius*2} ${link1_length - axel_offset*2}" rpy="0 0 0"/>
         <axis xyz="0 1 0"/>
@@ -84,5 +84,5 @@
     </joint>
     <!-- Top Link -->
-    <link name="BERT2_link3">
+    <link name="BERT2_link2">
         <collision>
             <origin xyz="0 0 ${link2_length/2 - axel_offset}" rpy="0 0 0"/>
@@ -145,5 +145,5 @@
         <material>Gazebo/Grey</material>
     </gazebo>
-    <gazebo reference="BERT2_link3">
+    <gazebo reference="BERT2_link2">
         <mu1>0.2</mu1>
         <mu2>0.2</mu2>

Commit message: Updated and cleaned up some more BERT stuff

File: src/ros_experimenting/models/BERT2.xacro (robot description, xacro)
@@ -3,16 +3,17 @@
     <!-- Constants for robot dimensions -->
     <xacro:property name="PI" value="3.1415926535897931"/>
+    <!-- Base Link -->
+    <xacro:property name="mass" value="5" />
+    <xacro:property name="height1" value="2" />
+    <xacro:property name="width" value="0.1" />
+    <!-- Middle Link -->
     <xacro:property name="link1_mass" value="2.35" />
+    <xacro:property name="link1_radius" value="0.05" />
+    <xacro:property name="link1_length" value="0.2735" />
+    <!-- Top Link -->
     <xacro:property name="link2_mass" value="3.0" />
-    <xacro:property name="link1_radius" value="0.05" />
     <xacro:property name="link2_radius" value="0.05" />
-    <xacro:property name="link1_length" value="0.2735" />
     <xacro:property name="link2_length" value="0.44" />
-    <xacro:property name="mass" value="5" />
     <xacro:property name="axel_offset" value="0.025" /> <!-- Space btw top of beam and the each joint -->
-    <xacro:property name="width" value="0.1" /> <!-- Square dimensions (widthxwidth) of beams -->
-    <xacro:property name="height1" value="2" /> <!-- Link 1 -->
-    <xacro:property name="height2" value="1" /> <!-- Link 2 -->
-    <xacro:property name="height3" value="1" /> <!-- Link 3 -->
     <!-- Make the robot's base immovable -->
     <link name="world"/>

Commit message: Adjusted the beam height of the robot

File: src/ros_experimenting/models/BERT2.xacro (robot description, xacro)
@@ -5,5 +5,5 @@
     <!-- Base Link -->
     <xacro:property name="mass" value="5" />
-    <xacro:property name="height1" value="2" />
+    <xacro:property name="height1" value="0.5" />
     <xacro:property name="width" value="0.1" />
     <!-- Middle Link -->

File: src/ros_experimenting/models/BERT2_robot.urdf (robot description, URDF)
Before this commit: robot BERT2_robot, 4 links, 3 joints
Links:
- link BERT2_baselink: geometry collision box size=0.1 0.1 0.5; visual box size=0.1 0.1 0.5
Joints:
- joint BERT2_joint1: origin xyz=0 0.1 1.975 rpy=0 0 0 -> xyz=0 0.1 0.475 rpy=0 0 0
